File: lm397breakout/lm397breakout.kicad_pcb (KiCad board)
At the start: 2 copper layers, 15.2 x 10.2 mm, 3 parts, among them J1 Conn_01x03, J2 Conn_01x03, U1 LM397

Commit message: rounded edges of breakout
Connections:
- net Net-(J1-Pad2) renamed GND
Routing:
- added copper zone on B.Cu, net GND
- added copper zone on F.Cu, net GND
Other:
- outline, holes or cut-outs redrawn
Changed lines of the file:
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@@
   (net 0 "")
   (net 1 "Net-(J1-Pad1)")
-  (net 2 "Net-(J1-Pad2)")
-  (net 3 "Net-(J1-Pad3)")
-  (net 4 "Net-(J2-Pad1)")
-  (net 5 "unconnected-(J2-Pad2)")
-  (net 6 "Net-(J2-Pad3)")
+  (net 2 "Net-(J1-Pad3)")
+  (net 3 "Net-(J2-Pad1)")
+  (net 4 "unconnected-(J2-Pad2)")
+  (net 5 "Net-(J2-Pad3)")
+  (net 6 "GND")
   (footprint "Connector_PinHeader_2.54mm:PinHeader_1x03_P2.54mm_Vertical" (layer "F.Cu")
     (at 157.48 99.06)
@@
     (fp_line (start 1.27 6.35) (end -1.27 6.35) (layer "F.Fab") (width 0.1))
     (pad "1" thru_hole rect (at 0 0) (size 1.7 1.7) (drill 1) (layers *.Cu *.Mask)
-      (net 4 "Net-(J2-Pad1)") (pinfunction "Pin_1") (pintype "passive"))
+      (net 3 "Net-(J2-Pad1)") (pinfunction "Pin_1") (pintype "passive"))
     (pad "2" thru_hole oval (at 0 2.54) (size 1.7 1.7) (drill 1) (layers *.Cu *.Mask)
-      (net 5 "unconnected-(J2-Pad2)") (pinfunction "Pin_2") (pintype "passive"))
+      (net 4 "unconnected-(J2-Pad2)") (pinfunction "Pin_2") (pintype "passive"))
     (pad "3" thru_hole oval (at 0 5.08) (size 1.7 1.7) (drill 1) (layers *.Cu *.Mask)
-      (net 6 "Net-(J2-Pad3)") (pinfunction "Pin_3") (pintype "passive"))
+      (net 5 "Net-(J2-Pad3)") (pinfunction "Pin_3") (pintype "passive"))
     (model "${KICAD6_3DMODEL_DIR}/Connector_PinHeader_2.54mm.3dshapes/PinHeader_1x03_P2.54mm_Vertical.wrl"
       (offset (xyz 0 0 0))
@@
       (net 1 "Net-(J1-Pad1)") (pinfunction "Pin_1") (pintype "passive"))
     (pad "2" thru_hole oval (at 0 2.54 180) (size 1.7 1.7) (drill 1) (layers *.Cu *.Mask)
-      (net 2 "Net-(J1-Pad2)") (pinfunction "Pin_2") (pintype "passive"))
+      (net 6 "GND") (pinfunction "Pin_2") (pintype "passive"))
     (pad "3" thru_hole oval (at 0 5.08 180) (size 1.7 1.7) (drill 1) (layers *.Cu *.Mask)
-      (net 3 "Net-(J1-Pad3)") (pinfunction "Pin_3") (pintype "passive"))
+      (net 2 "Net-(J1-Pad3)") (pinfunction "Pin_3") (pintype "passive"))
     (model "${KICAD6_3DMODEL_DIR}/Connector_PinHeader_2.54mm.3dshapes/PinHeader_1x03_P2.54mm_Vertical.wrl"
       (offset (xyz 0 0 0))
@@
     (fp_line (start 0.8 1.45) (end -0.8 1.45) (layer "F.Fab") (width 0.1))
     (pad "1" smd roundrect (at -1.1375 -0.95) (size 1.325 0.6) (layers "F.Cu" "F.Paste" "F.Mask") (roundrect_rratio 0.25)
-      (net 3 "Net-(J1-Pad3)") (pinfunction "-") (pintype "input"))
+      (net 2 "Net-(J1-Pad3)") (pinfunction "-") (pintype "input"))
     (pad "2" smd roundrect (at -1.1375 0) (size 1.325 0.6) (layers "F.Cu" "F.Paste" "F.Mask") (roundrect_rratio 0.25)
-      (net 2 "Net-(J1-Pad2)") (pinfunction "V-") (pintype "power_in"))
+      (net 6 "GND") (pinfunction "V-") (pintype "power_in"))
     (pad "3" smd roundrect (at -1.1375 0.95) (size 1.325 0.6) (layers "F.Cu" "F.Paste" "F.Mask") (roundrect_rratio 0.25)
       (net 1 "Net-(J1-Pad1)") (pinfunction "+") (pintype "input"))
     (pad "4" smd roundrect (at 1.1375 0.95) (size 1.325 0.6) (layers "F.Cu" "F.Paste" "F.Mask") (roundrect_rratio 0.25)
-      (net 6 "Net-(J2-Pad3)") (pintype "open_collector"))
+      (net 5 "Net-(J2-Pad3)") (pintype "open_collector"))
     (pad "5" smd roundrect (at 1.1375 -0.95) (size 1.325 0.6) (layers "F.Cu" "F.Paste" "F.Mask") (roundrect_rratio 0.25)
-      (net 4 "Net-(J2-Pad1)") (pinfunction "V+") (pintype "power_in"))
+      (net 3 "Net-(J2-Pad1)") (pinfunction "V+") (pintype "power_in"))
     (model "${KICAD6_3DMODEL_DIR}/Package_TO_SOT_SMD.3dshapes/SOT-23-5.wrl"
       (offset (xyz 0 0 0))
@@
     )
   )
-  (gr_line (start 144.78 96.52) (end 144.78 106.68) (layer "Edge.Cuts") (width 0.1))
-  (gr_line (start 160.02 96.52) (end 160.02 106.68) (layer "Edge.Cuts") (width 0.1))
-  (gr_line (start 160.02 106.68) (end 144.78 106.68) (layer "Edge.Cuts") (width 0.1))
-  (gr_line (start 144.78 96.52) (end 160.02 96.52) (layer "Edge.Cuts") (width 0.1))
+  (gr_line (start 158.75 106.68) (end 146.05 106.68) (layer "Edge.Cuts") (width 0.1))
+  (gr_line (start 160.02 97.79) (end 160.02 105.41) (layer "Edge.Cuts") (width 0.1))
+  (gr_arc (start 144.78 97.79) (mid 145.151974 96.891974) (end 146.05 96.52) (layer "Edge.Cuts") (width 0.1))
+  (gr_arc (start 160.02 105.41) (mid 159.648026 106.308026) (end 158.75 106.68) (layer "Edge.Cuts") (width 0.1))
+  (gr_line (start 144.78 105.41) (end 144.78 97.79) (layer "Edge.Cuts") (width 0.1))
+  (gr_line (start 146.05 96.52) (end 158.75 96.52) (layer "Edge.Cuts") (width 0.1))
+  (gr_arc (start 146.05 106.68) (mid 145.151974 106.308026) (end 144.78 105.41) (layer "Edge.Cuts") (width 0.1))
+  (gr_arc (start 158.75 96.52) (mid 159.648026 96.891974) (end 160.02 97.79) (layer "Edge.Cuts") (width 0.1))
   (segment (start 149.5725 104.14) (end 151.2625 102.45) (width 0.4) (layer "F.Cu") (net 1))
   (segment (start 147.32 104.14) (end 149.5725 104.14) (width 0.4) (layer "F.Cu") (net 1))
-  (segment (start 151.1625 101.6) (end 151.2625 101.5) (width 0.25) (layer "F.Cu") (net 2))
-  (segment (start 147.42 101.5) (end 147.32 101.6) (width 0.4) (layer "F.Cu") (net 2))
-  (segment (start 151.2625 101.5) (end 147.42 101.5) (width 0.4) (layer "F.Cu") (net 2))
-  (segment (start 149.86 99.06) (end 151.2625 100.4625) (width 0.4) (layer "F.Cu") (net 3))
-  (segment (start 147.32 99.06) (end 149.86 99.06) (width 0.4) (layer "F.Cu") (net 3))
-  (segment (start 151.2625 100.4625) (end 151.2625 100.55) (width 0.4) (layer "F.Cu") (net 3))
-  (segment (start 153.5375 100.55) (end 153.5375 100.4625) (width 0.4) (layer "F.Cu") (net 4))
-  (segment (start 153.5375 100.4625) (end 154.94 99.06) (width 0.4) (layer "F.Cu") (net 4))
-  (segment (start 154.94 99.06) (end 157.48 99.06) (width 0.4) (layer "F.Cu") (net 4))
-  (segment (start 153.5375 102.7375) (end 154.94 104.14) (width 0.4) (layer "F.Cu") (net 6))
-  (segment (start 154.94 104.14) (end 157.48 104.14) (width 0.4) (layer "F.Cu") (net 6))
-  (segment (start 153.5375 102.45) (end 153.5375 102.7375) (width 0.4) (layer "F.Cu") (net 6))
+  (segment (start 149.86 99.06) (end 151.2625 100.4625) (width 0.4) (layer "F.Cu") (net 2))
+  (segment (start 147.32 99.06) (end 149.86 99.06) (width 0.4) (layer "F.Cu") (net 2))
+  (segment (start 151.2625 100.4625) (end 151.2625 100.55) (width 0.4) (layer "F.Cu") (net 2))
+  (segment (start 153.5375 100.55) (end 153.5375 100.4625) (width 0.4) (layer "F.Cu") (net 3))
+  (segment (start 153.5375 100.4625) (end 154.94 99.06) (width 0.4) (layer "F.Cu") (net 3))
+  (segment (start 154.94 99.06) (end 157.48 99.06) (width 0.4) (layer "F.Cu") (net 3))
+  (segment (start 153.5375 102.7375) (end 154.94 104.14) (width 0.4) (layer "F.Cu") (net 5))
+  (segment (start 154.94 104.14) (end 157.48 104.14) (width 0.4) (layer "F.Cu") (net 5))
+  (segment (start 153.5375 102.45) (end 153.5375 102.7375) (width 0.4) (layer "F.Cu") (net 5))
+  (segment (start 151.1625 101.6) (end 151.2625 101.5) (width 0.25) (layer "F.Cu") (net 6))
+  (segment (start 147.42 101.5) (end 147.32 101.6) (width 0.4) (layer "F.Cu") (net 6))
+  (segment (start 151.2625 101.5) (end 147.42 101.5) (width 0.4) (layer "F.Cu") (net 6))
+  (zone (net 6) (net_name "GND") (layer "F.Cu") (hatch edge 0.508)
+    (connect_pads (clearance 0.508))
+    (min_thickness 0.254) (filled_areas_thickness no)
+    (fill yes (thermal_gap 0.508) (thermal_bridge_width 0.508))
+    (polygon
+      (pts
+        (xy 160.02 106.68)
+        (xy 144.78 106.68)
+        (xy 144.78 96.52)
+        (xy 160.02 96.52)
+      )
+    )
+  )
+  (zone (net 6) (net_name "GND") (layer "B.Cu") (hatch edge 0.508)
+    (connect_pads (clearance 0.508))
+    (min_thickness 0.254) (filled_areas_thickness no)
+    (fill yes (thermal_gap 0.508) (thermal_bridge_width 0.508))
+    (polygon
+      (pts
+        (xy 160.02 106.68)
+        (xy 144.78 106.68)
+        (xy 144.78 96.52)
+        (xy 160.02 96.52)
+      )
+    )
+  )
 )
