File: lm397breakout/lm397breakout.kicad_sch (KiCad schematic)
At the start: 3 parts

Commit message: rounded edges of breakout
Parts:
- gave numbers to parts that had none: 3
Connections:
- net GND: now reaches J1.2 (Pin_2), U1.2 (V-)
Changed lines of the file:
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@@
 (kicad_sch (version 20211123) (generator eeschema)
   (paper "A4")
+  (junction (at 116.84 64.77) (diameter 0) (color 0 0 0 0)
+  )
   (wire (pts (xy 109.22 54.61) (xy 109.22 59.69))
     (stroke (width 0) (type default) (color 0 0 0 0))
@@
   (symbol (lib_id "Connector_Generic:Conn_01x03") (at 140.97 57.15 0) (unit 1)
     (in_bom yes) (on_board yes) (fields_autoplaced)
-    (property "Reference" "J?" (id 0) (at 143.51 55.8799 0)
+    (property "Reference" "J2" (id 0) (at 143.51 55.8799 0)
       (effects (font (size 1.27 1.27)) (justify left))
     )
@@
     (pin "3")
   )
+  (symbol (lib_id "power:GND") (at 116.84 64.77 0) (unit 1)
+    (in_bom yes) (on_board yes) (fields_autoplaced)
+    (property "Reference" "#PWR?" (id 0) (at 116.84 71.12 0)
+      (effects (font (size 1.27 1.27)) hide)
+    )
+    (property "Value" "GND" (id 1) (at 116.84 69.85 0))
+    (property "Footprint" "" (id 2) (at 116.84 64.77 0)
+      (effects (font (size 1.27 1.27)) hide)
+    )
+    (property "Datasheet" "" (id 3) (at 116.84 64.77 0)
+      (effects (font (size 1.27 1.27)) hide)
+    )
+    (pin "1")
+  )
   (symbol (lib_id "Comparator:LM397") (at 119.38 57.15 0) (unit 1)
     (in_bom yes) (on_board yes)
-    (property "Reference" "U?" (id 0) (at 119.38 43.18 0))
+    (property "Reference" "U1" (id 0) (at 119.38 43.18 0))
     (property "Value" "LM397" (id 1) (at 119.38 46.99 0))
     (property "Footprint" "Package_TO_SOT_SMD:SOT-23-5" (id 2) (at 120.65 72.39 0)
@@
   (symbol (lib_id "Connector_Generic:Conn_01x03") (at 101.6 57.15 180) (unit 1)
     (in_bom yes) (on_board yes) (fields_autoplaced)
-    (property "Reference" "J?" (id 0) (at 101.6 48.26 0))
+    (property "Reference" "J1" (id 0) (at 101.6 48.26 0))
     (property "Value" "Conn_01x03" (id 1) (at 101.6 50.8 0))
     (property "Footprint" "" (id 2) (at 101.6 57.15 0)
@@
   )
   (symbol_instances
-    (path "/323e6016-9796-4740-b49a-d38b5ab6284c"
-      (reference "J?") (unit 1) (value "Conn_01x03") (footprint "Connector_PinHeader_2.54mm:PinHeader_1x03_P2.54mm_Vertical")
+    (path "/a1094997-411b-4bce-8143-00b976bc3c7d"
+      (reference "#PWR?") (unit 1) (value "GND") (footprint "")
     )
     (path "/fa7965c8-12aa-4fc0-aeaa-c50d00202f9f"
-      (reference "J?") (unit 1) (value "Conn_01x03") (footprint "Connector_PinHeader_2.54mm:PinHeader_1x03_P2.54mm_Vertical")
+      (reference "J1") (unit 1) (value "Conn_01x03") (footprint "Connector_PinHeader_2.54mm:PinHeader_1x03_P2.54mm_Vertical")
+    )
+    (path "/323e6016-9796-4740-b49a-d38b5ab6284c"
+      (reference "J2") (unit 1) (value "Conn_01x03") (footprint "Connector_PinHeader_2.54mm:PinHeader_1x03_P2.54mm_Vertical")
     )
     (path "/f24c34e4-33be-4b94-a26a-1d05fba4c36c"
-      (reference "U?") (unit 1) (value "LM397") (footprint "Package_TO_SOT_SMD:SOT-23-5")
+      (reference "U1") (unit 1) (value "LM397") (footprint "Package_TO_SOT_SMD:SOT-23-5")
     )
   )
